File: Hardware/eeprom_burner_arduino_shield_eagle/eeprom_burner.sch (EAGLE design)
At the start: 5 parts, among them IC2 74LS595N, IC3 74LS595N

Commit message: updated board layout
Parts:
- added JP1: 256 / 16 switch 1, pinhead:PINHD-1X3
- added JP2: 256 / 16 switch 2, pinhead:PINHD-1X3
- added LED1, LED2: (no value), led:LED3MM
- added R1, R2: 470, resistor:R-EU_0204/7
- U$1: value ARDUINOUNO -> ARDUINO-NODIM; device adafruit:ARDUINOUNO -> adafruit:ARDUINO-NODIM
Connections:
- new net A11: IC3A.QD, JP2.1
- new net A13: IC3A.QF, JP1.1
- new net N$28: LED2.A, R2.2
- new net PIN23: 28C256A.A11, JP2.2
- new net PIN26: 28C256A.A13, JP1.2
- new net WE: 28C256A.!WE, JP2.3, U$1.A5
- net GND: now also LED1.C, LED2.C
- net N$1: now also R2.1, U$1.D12; no longer 28C256A.!WE, U$1.A5
- net N$24: now also R1.1, U$1.D13; no longer 28C256A.A11, IC3A.QD
- net N$26: now also LED1.A, R1.2; no longer 28C256A.A13, IC3A.QF
- net VCC: now also JP1.3
Other:
- moved on the sheet: IC2, IC3
